Commit message: work in progress. DTD complains about robot tag

File: uwsim/data/scenes/cirs.xml.xacro (robot description, xacro)
@@ -2,283 +2,51 @@
 <!DOCTYPE UWSimScene SYSTEM "UWSimScene.dtd">
 <robot xmlns:xacro="http://www.ros.org/wiki/xacro" name="girona500">
-<xacro:include filename="params_base.xacro" />
-<xacro:include filename="common.xacro" />
-<UWSimScene>
-  <oceanState>
-    <windx> 0.04 </windx>
-    <windy> 0.04 </windy>
-    <windSpeed> 12 </windSpeed>
-    <depth> 1000 </depth>
-    <reflectionDamping> 0.35 </reflectionDamping>
-    <waveScale> 1e-7 </waveScale>
-    <isNotChoppy> 0 </isNotChoppy>
-    <choppyFactor> 2.5 </choppyFactor>
-    <crestFoamHeight> 2.2 </crestFoamHeight>
-    <oceanSurfaceHeight> 0 </oceanSurfaceHeight>
-    <fog>
-      <density> 0.1</density>
-      <color>
-	<r>0</r>
-	<g>0.05</g>
-	<b>0.3</b>
-      </color>
-    </fog>
-    <color>
-      <r>0.0</r>
-      <g>0.05</g>
-      <b>0.3</b>
-    </color>
-    <attenuation>
-      <r>0.015</r>
-      <g>0.0075 </g>
-      <b> 0.005 </b>
-    </attenuation>
-  </oceanState>
-  <simParams>
-    <disableShaders> 0 </disableShaders>
-    <resw> 800 </resw>
-    <resh> 600 </resh>
-    <offsetp>
-      <x>0</x>
-      <y>0</y>
-      <z>0</z>
-    </offsetp>
-    <offsetr>
-      <x> 3.14</x>
-      <y> 0</y>
-      <z> -1.57 </z>
-    </offsetr>
-    <enablePhysics> 1 </enablePhysics>
-    <showTrajectory>
-      <target>girona500</target>
-    </showTrajectory>
-  </simParams>
-  <camera>
-    <freeMotion> 1 </freeMotion>
-    <objectToTrack>girona500/base_link</objectToTrack>
-    <fov> 60 </fov>
-    <aspectRatio> 1.33 </aspectRatio>
-    <near> 1 </near>
-    <far> 10000 </far>
-    <position>
-      <x>-5</x>
-      <y>-5 </y>
-      <z>8 </z>
-    </position>
-    <lookAt>
-      <x>0</x>
-      <y>0 </y>
-      <z>0 </z>
-    </lookAt>
-  </camera>
-  <vehicle>
-    <name>girona500</name>
-    <file>data/scenes/g500ARM5.urdf</file>
-    <jointValues>
-      <joint> 0 </joint>
-      <joint> 0</joint>
-      <joint> 2.2 </joint>
-      <joint> 0 </joint>
-      <joint>0.3 </joint>
-    </jointValues>
-    <position>
-      <x> 0.2</x>
-      <y> 0 </y>
-      <z> 2.0 </z>
-    </position>
-    <orientation>
-      <r>0</r>
-      <p>0</p>
-      <y>0</y>
-    </orientation>
-    <xacro:bowtech_stereo_pair/>
-    <xacro:range_sensor name="sonar" link="part0" x="-0.3" y="0" z="0" roll="0" pitch="${M_PI/2}" yaw="0" range="10" />
-    <xacro:imu_sensor name="imu" link="base_link" x="0" y="0" z="0" roll="0" pitch="0" yaw="${M_PI}" std_dev="0.00000001" />
-    <xacro:pressure_sensor name="pressure_sensor" link="base_link" x="0" y="0" z="0.2" roll="0" pitch="0" yaw="0" std_dev="0.02" />
-    <xacro:gps_sensor name="gps_sensor" link="base_link" x="0" y="0" z="0.2" roll="0" pitch="0" yaw="0" std_dev="0.00005" />
-    <xacro:dvl_sensor name="dvl_sensor" link="base_link" x="-0.75" y="0" z="0.2" roll="0" pitch="0" yaw="3.9269908169872414" std_dev="0.0015" />
-    <xacro:depth_camera_sensor name="depth_camera" link="part0" resw="320" resh="240" f="257.986" x="-0.2" y="0.1" z="0" roll="0" pitch="0" yaw="${M_PI/2}"/>
-    <multibeamSensor>
-      <name>multibeam</name>
-      <relativeTo>part0</relativeTo>
+  <xacro:include filename="params_base.xacro" />
+  <xacro:include filename="common.xacro" />
+  <UWSimScene>
+    <xacro:default_ocean/>
+    <xacro:default_simulation_params/>
+    <camera>
+      <freeMotion> 1 </freeMotion>
+      <objectToTrack>girona500/base_link</objectToTrack>
+      <fov> 60 </fov>
+      <aspectRatio> 1.33 </aspectRatio>
+      <near> 1 </near>
+      <far> 10000 </far>
       <position>
-        <x>-0.2</x>
-        <y> 0.1 </y>
-        <z> 0 </z>
+        <x>-5</x>
+        <y>-5 </y>
+        <z>8 </z>
       </position>
-      <orientation>
-        <r>0</r>
-        <p>0</p>
-        <y>3.14 </y>
-      </orientation>
-      <initAngle>-60</initAngle>
-      <finalAngle>60</finalAngle>
-      <angleIncr>0.1</angleIncr>
-      <range>10</range>
-    </multibeamSensor>
-    <simulatedDevices>
-      <echo>
-        <name>g500_echo1</name>
-        <info>Echo example 1</info>
-      </echo>
-    </simulatedDevices>
-    <echo>
-      <name>g500_echo2</name>
-      <info>Echo example 2</info>
-    </echo>
-    <ForceSensor>
-      <name>ForceG500</name>
-      <target>base_link</target>
-      <offsetp>
-        <x>-0.2</x>
-        <y>0.75</y>
-        <z>0</z>
-      </offsetp>
-      <offsetr>
-        <x>-1.57</x>
-        <y>0</y>
-        <z>3.14</z>
-      </offsetr>
-    </ForceSensor>
-  </vehicle>
-  <object>
-    <name>terrain</name>
-    <file>terrain/CIRS/cirs_trident.osg</file>
-    <position>
-      <x> 0</x>
-      <y> 0 </y>
-      <z> 0 </z>
-    </position>
-    <orientation>
-      <r>0</r>
-      <p>0</p>
-      <y>0</y>
-    </orientation>
-    <offsetp>
-      <x>-1.5</x>
-      <y>-3.0</y>
-      <z>0</z>
-    </offsetp>
-    <offsetr>
-      <x> 3.1415</x>
-      <y> 0</y>
-      <z> -1.57 </z>
-    </offsetr>
-    <physics>
-      <mass> 0 </mass>
-      <collisionShapeType> trimesh </collisionShapeType>
-    </physics>
-  </object>
-  <object>
-    <name> blackbox </name>
-    <file> objects/blackbox_uib_trimesh.osg  </file>
-    <position>
-      <x> 0</x>
-      <y> 0 </y>
-      <z> 4.7 </z>
-    </position>
-    <orientation>
-      <r>0</r>
-      <p>3.1415</p>
-      <y>0</y>
-    </orientation>
-    <physics>
-      <mass> 15 </mass>
-      <inertia>
-        <x> 0</x>
-        <y> 0 </y>
-        <z> 0 </z>
-      </inertia>
-      <collisionShapeType> box </collisionShapeType>
-    </physics>
-  </object>
-  <rosInterfaces>
-    <ROSOdomToPAT>
-      <topic> /dataNavigator </topic>
-      <vehicleName> girona500 </vehicleName>
-    </ROSOdomToPAT>
-    <WorldToROSTF>
-      <rootName> world </rootName>
-      <enableObjects> 1 </enableObjects>
-      <rate>10</rate>
-    </WorldToROSTF>
-    <ArmToROSJointState>
-	<topic>/uwsim/joint_state</topic>
-	<vehicleName> girona500 </vehicleName>
-    </ArmToROSJointState>
-    <ROSJointStateToArm>
-	<topic>/uwsim/joint_state_command</topic>
-	<vehicleName> girona500 </vehicleName>
-    </ROSJointStateToArm>
-    <VirtualCameraToROSImage>
-      <cameraName>bowtech1</cameraName>
-      <imageTopic> /uwsim/camera1 </imageTopic>
-      <infoTopic> /uwsim/camera1_info </infoTopic>
-    </VirtualCameraToROSImage>
-    <ROSTwistToPAT>
-      <topic> /g500/twist</topic>
-      <vehicleName> girona500 </vehicleName>
-    </ROSTwistToPAT>
-    <RangeSensorToROSRange>
-      <name>sonar</name>
-      <topic> /uwsim/g500/range </topic>
-      <rate>10</rate>
-    </RangeSensorToROSRange>
-    <ROSPoseToPAT>
-      <topic> /g500/pose</topic>
-      <vehicleName> girona500 </vehicleName>
-    </ROSPoseToPAT>
-    <ImuToROSImu>
-      <name>imu</name>
-      <topic>g500/imu</topic>
-      <rate>20</rate>
-    </ImuToROSImu>
-    <PressureSensorToROS>
-      <name>pressureSensor</name>
-      <topic>g500/pressure</topic>
-      <rate>5</rate>
-    </PressureSensorToROS>
-    <GPSSensorToROS>
-      <name>GPSSensor</name>
-      <topic>g500/gps</topic>
-      <rate>1</rate>
-    </GPSSensorToROS>
-    <DVLSensorToROS>
-      <name>DVLSensor</name>
-      <topic>g500/dvl</topic>
-      <rate>5</rate>
-    </DVLSensorToROS>
-    <RangeImageSensorToROSImage>
-      <cameraName>rangeImage</cameraName>
-      <imageTopic> /uwsim/rangecamera </imageTopic>
-      <infoTopic> /uwsim/rangecamera_info </infoTopic>
-    </RangeImageSensorToROSImage>
-    <multibeamSensorToLaserScan>
-      <name>multibeam</name>
-      <topic>g500/multibeam</topic>
-    </multibeamSensorToLaserScan>
-    <SimulatedDeviceROS>
-      <echoROS>
-        <name>g500_echo1</name>
-        <topic>g500/echo1</topic>
-        <rate>1</rate>
-      </echoROS>
-    </SimulatedDeviceROS>
-    <contactSensorToROS>
+      <lookAt>
+        <x>0</x>
+        <y>0 </y>
+        <z>0 </z>
+      </lookAt>
+    </camera>
+    <vehicle>
       <name>girona500</name>
-      <topic>g500/contactSensor</topic>
-      <rate> 100 </rate>
-    </contactSensorToROS>
-    <echoROS>
-      <name>g500_echo2</name>
-      <topic>g500/echo2</topic>
-      <rate>1</rate>
-    </echoROS>
-    <ForceSensorROS>
-      <name>ForceG500</name>
-      <topic>g500/ForceSensor</topic>
-      <rate>100</rate>
-    </ForceSensorROS>
-  </rosInterfaces>
-</UWSimScene>
+      <file>data/scenes/g500ARM5.urdf</file>
+      <jointValues>
+        <joint> 0 </joint>
+        <joint> 0</joint>
+        <joint> 2.2 </joint>
+        <joint> 0 </joint>
+        <joint>0.3 </joint>
+      </jointValues>
+      <xacro:pose x="0.2" y="0" z="2.0" roll="0" pitch="0" yaw="0" />
+      <xacro:bowtech_stereo_pair/>
+      <xacro:range_sensor name="sonar" link="part0" x="-0.3" y="0" z="0" roll="0" pitch="${M_PI/2}" yaw="0" range="10" />
+      <xacro:imu_sensor name="imu" link="base_link" x="0" y="0" z="0" roll="0" pitch="0" yaw="${M_PI}" std_dev="0.00000001" />
+      <xacro:pressure_sensor name="pressure_sensor" link="base_link" x="0" y="0" z="0.2" roll="0" pitch="0" yaw="0" std_dev="0.02" />
+      <xacro:gps_sensor name="gps_sensor" link="base_link" x="0" y="0" z="0.2" roll="0" pitch="0" yaw="0" std_dev="0.00005" />
+      <xacro:dvl_sensor name="dvl_sensor" link="base_link" x="-0.75" y="0" z="0.2" roll="0" pitch="0" yaw="3.9269908169872414" std_dev="0.0015" />
+      <xacro:depth_camera_sensor name="depth_camera" link="part0" resw="320" resh="240" f="257.986" x="-0.2" y="0.1" z="0" roll="0" pitch="0" yaw="${M_PI/2}"/>
+      <xacro:multibeam_sensor name="multibeam_sensor" link="part0" x="-0.2" y="0.1" z="0" roll="0" pitch="0" yaw="M_PI" init_angle="-60" final_angle="60" incr="0.1" range="10" />
+      <xacro:force_sensor name="force_sensor" target="base_link" offsetpx="-0.2" offsetpy="0.75" offsetpz="0" offsetrx="${-M_PI/2}" offsetry="0" offsetrz="${M_PI}" />
+    </vehicle>
+    <xacro:add_object name="terrain" file="terrain/CIRS/cirs_trident.osg" offsetpx="-1.5" offsetpy="-3.0" offsetpz="0" offsetrx="3.1415" offsetry="0" offsetrz="-1.57" mass="0" mesh="trimesh" />
+    <xacro:add_object name="blackbox" file="objects/blackbox_uib_trimesh.osg" offsetpx="0" offsetpy="0" offsetpz="4.7" offsetrx="0" offsetry="3.1415" offsetrz="0" mass="15" mesh="box" />
+    <xacro:ros_interfaces/>
+  </UWSimScene>
 </robot>

File: uwsim/data/scenes/common.xacro (robot description, xacro)
@@ -1,6 +1,58 @@
 <?xml version="1.0"?>
 <robot xmlns:xacro="http://www.ros.org/wiki/xacro" name="girona500">
-	<xacro:macro name="pose" params="link x y z roll pitch yaw">
-    <relativeTo> ${link} </relativeTo>
+	<xacro:macro name="default_ocean">
+		<oceanState>
+	      <windx> 0.04 </windx>
+	      <windy> 0.04 </windy>
+	      <windSpeed> 12 </windSpeed>
+	      <depth> 1000 </depth>
+	      <reflectionDamping> 0.35 </reflectionDamping>
+	      <waveScale> 1e-7 </waveScale>
+	      <isNotChoppy> 0 </isNotChoppy>
+	      <choppyFactor> 2.5 </choppyFactor>
+	      <crestFoamHeight> 2.2 </crestFoamHeight>
+	      <oceanSurfaceHeight> 0 </oceanSurfaceHeight>
+	      <fog>
+	        <density> 0.1</density>
+	        <color>
+	          <r>0</r>
+	          <g>0.05</g>
+	          <b>0.3</b>
+	        </color>
+	      </fog>
+	      <color>
+	        <r>0.0</r>
+	        <g>0.05</g>
+	        <b>0.3</b>
+	      </color>
+	      <attenuation>
+	        <r>0.015</r>
+	        <g>0.0075 </g>
+	        <b> 0.005 </b>
+	      </attenuation>
+	    </oceanState>
+	</xacro:macro>
+	<xacro:macro name="default_simulation_params">
+    <simParams>
+      <disableShaders> 0 </disableShaders>
+      <resw> 800 </resw>
+      <resh> 600 </resh>
+      <offsetp>
+        <x>0</x>
+        <y>0</y>
+        <z>0</z>
+      </offsetp>
+      <offsetr>
+        <x> 3.14</x>
+        <y> 0</y>
+        <z> -1.57 </z>
+      </offsetr>
+      <enablePhysics> 1 </enablePhysics>
+      <showTrajectory>
+        <target>girona500</target>
+      </showTrajectory>
+    </simParams>
+  </xacro:macro>
+	<xacro:macro name="pose" params="x y z roll pitch yaw">
     <position>
       <x> ${x} </x>
@@ -14,8 +66,12 @@
     </orientation>
   </xacro:macro>
+	<xacro:macro name="relative_pose" params="link x y z roll pitch yaw">
+    <relativeTo> ${link} </relativeTo>
+    <xacro:pose x="${x}" y="${y}" z="${z}" roll="${roll}" pitch="${pitch}" yaw="${yaw}" />
+  </xacro:macro>
   <xacro:macro name="camera_sensor" params="name link resw resh f x y z roll pitch yaw">
     <virtualCamera>
       <name> ${name} </name>
-      <xacro:pose link="${link}" x="${x}" y="${y}" z="${z}" roll="${roll}" pitch="${pitch}" yaw="${yaw}" />
+      <xacro:relative_pose link="${link}" x="${x}" y="${y}" z="${z}" roll="${roll}" pitch="${pitch}" yaw="${yaw}" />
       <resw> ${resw} </resw>
       <resh> ${resh} </resh>
@@ -34,5 +90,5 @@
     <virtualRangeImage>
       <name> ${name} </name>
-      <xacro:pose link="${link}" x="${x}" y="${y}" z="${z}" roll="${roll}" pitch="${pitch}" yaw="${yaw}" />
+      <xacro:relative_pose link="${link}" x="${x}" y="${y}" z="${z}" roll="${roll}" pitch="${pitch}" yaw="${yaw}" />
       <resw> ${resw} </resw>
       <resh> ${resh} </resh>
@@ -51,5 +107,5 @@
     <rangeSensor>
       <name> ${name} </name>
-      <xacro:pose link="${link}" x="${x}" y="${y}" z="${z}" roll="${roll}" pitch="${pitch}" yaw="${yaw}" />
+      <xacro:relative_pose link="${link}" x="${x}" y="${y}" z="${z}" roll="${roll}" pitch="${pitch}" yaw="${yaw}" />
       <range> ${range} </range>
       <visible> 0 </visible>
@@ -59,5 +115,5 @@
     <imu>
       <name> ${name} </name>
-      <xacro:pose link="${link}" x="${x}" y="${y}" z="${z}" roll="${roll}" pitch="${pitch}" yaw="${yaw}" />
+      <xacro:relative_pose link="${link}" x="${x}" y="${y}" z="${z}" roll="${roll}" pitch="${pitch}" yaw="${yaw}" />
       <std> ${std_dev} </std>
     </imu>
@@ -66,5 +122,5 @@
     <pressureSensor>
       <name> ${name} </name>
-      <xacro:pose link="${link}" x="${x}" y="${y}" z="${z}" roll="${roll}" pitch="${pitch}" yaw="${yaw}" />
+      <xacro:relative_pose link="${link}" x="${x}" y="${y}" z="${z}" roll="${roll}" pitch="${pitch}" yaw="${yaw}" />
       <std> ${std_dev} </std>
     </pressureSensor>
@@ -73,5 +129,5 @@
     <gpsSensor>
       <name> ${name} </name>
-      <xacro:pose link="${link}" x="${x}" y="${y}" z="${z}" roll="${roll}" pitch="${pitch}" yaw="${yaw}" />
+      <xacro:relative_pose link="${link}" x="${x}" y="${y}" z="${z}" roll="${roll}" pitch="${pitch}" yaw="${yaw}" />
       <std> ${std_dev} </std>
     </gpsSensor>
@@ -80,5 +136,5 @@
     <dvlSensor>
       <name> ${name} </name>
-      <xacro:pose link="${link}" x="${x}" y="${y}" z="${z}" roll="${roll}" pitch="${pitch}" yaw="${yaw}" />
+      <xacro:relative_pose link="${link}" x="${x}" y="${y}" z="${z}" roll="${roll}" pitch="${pitch}" yaw="${yaw}" />
       <std> ${std_dev} </std>
     </dvlSensor>
@@ -88,3 +144,152 @@
     <xacro:camera_sensor name="bowtech2" link="part0" resw="320" resh="240" f="160" x="-0.2" y="+0.1" z="0" roll="0" pitch="0" yaw="${M_PI/2}"/>
   </xacro:macro>
+  <xacro:macro name="multibeam_sensor" params="name link x y z roll pitch yaw init_angle final_angle incr range">
+    <multibeamSensor>
+      <name> ${name} </name>
+      <xacro:relative_pose link="${link}" x="${x}" y="${y}" z="${z}" roll="${roll}" pitch="${pitch}" yaw="${yaw}" />
+      <initAngle>${init_angle}</initAngle>
+      <finalAngle>${final_angle}</finalAngle>
+      <angleIncr>${incr}</angleIncr>
+      <range>${range}</range>
+    </multibeamSensor>
+  </xacro:macro>
+  <xacro:macro name="force_sensor" params="name target offsetpx offsetpy offsetpz offsetrx offsetry offsetrz">
+    <ForceSensor>
+      <name> ${name} </name>
+      <target> ${target} </target>
+      <offsetp>
+        <x>${offsetpx}</x>
+        <y>${offsetpy}</y>
+        <z>${offsetpz}</z>
+      </offsetp>
+      <offsetr>
+        <x>${offsetrx}</x>
+        <y>${offsetry}</y>
+        <z>${offsetrz}</z>
+      </offsetr>
+    </ForceSensor>
+  </xacro:macro>
+  <xacro:macro name="default_position">
+  	<position>
+      <x> 0 </x>
+      <y> 0 </y>
+      <z> 0 </z>
+    </position>
+    <orientation>
+      <r> 0 </r>
+      <p> 0 </p>
+      <y> 0 </y>
+    </orientation>
+  </xacro:macro>
+  <xacro:macro name="add_object" params="name file offsetpx offsetpy offsetpz offsetrx offsetry offsetrz mass mesh">
+  	<object>
+	    <name>${name}</name>
+	    <file>${file}</file>
+	    <xacro:default_position/>
+	    <offsetp>
+        <x>${offsetpx}</x>
+        <y>${offsetpy}</y>
+        <z>${offsetpz}</z>
+      </offsetp>
+      <offsetr>
+        <x>${offsetrx}</x>
+        <y>${offsetry}</y>
+        <z>${offsetrz}</z>
+      </offsetr>
+	    <physics>
+	      <mass> ${mass} </mass>
+	      <collisionShapeType> ${mesh} </collisionShapeType>
+	    </physics>
+  	</object>
+  </xacro:macro>
+  <xacro:macro name="ros_interfaces">
+  	<rosInterfaces>
+  		<ROSOdomToPAT>
+  			<topic> /${ns}/dataNavigator </topic>
+  			<vehicleName> ${vehicle_name} </vehicleName>
+  		</ROSOdomToPAT>
+  		<WorldToROSTF>
+  			<rootName> world </rootName>
+  			<enableObjects> 1 </enableObjects>
+  			<rate>10</rate>
+  		</WorldToROSTF>
+  		<ArmToROSJointState>
+  			<topic>/${ns}/joint_state</topic>
+  			<vehicleName> ${vehicle_name} </vehicleName>
+  		</ArmToROSJointState>
+  		<ROSJointStateToArm>
+  			<topic>/${ns}/joint_state_command</topic>
+  			<vehicleName> ${vehicle_name} </vehicleName>
+  		</ROSJointStateToArm>
+  		<VirtualCameraToROSImage>
+  			<cameraName>bowtech1</cameraName>
+  			<imageTopic> /${ns}/camera1 </imageTopic>
+  			<infoTopic> /${ns}/camera1_info </infoTopic>
+  		</VirtualCameraToROSImage>
+  		<ROSTwistToPAT>
+  			<topic> /${ns}/twist</topic>
+  			<vehicleName> ${vehicle_name} </vehicleName>
+  		</ROSTwistToPAT>
+  		<RangeSensorToROSRange>
+  			<name>sonar</name>
+  			<topic> /${ns}/range </topic>
+  			<rate>10</rate>
+  		</RangeSensorToROSRange>
+  		<ROSPoseToPAT>
+  			<topic> /${ns}/pose</topic>
+  			<vehicleName> ${vehicle_name} </vehicleName>
+  		</ROSPoseToPAT>
+  		<ImuToROSImu>
+  			<name>imu</name>
+  			<topic>/${ns}/imu</topic>
+  			<rate>20</rate>
+  		</ImuToROSImu>
+  		<PressureSensorToROS>
+  			<name>pressure_sensor</name>
+  			<topic>/${ns}/pressure</topic>
+  			<rate>5</rate>
+  		</PressureSensorToROS>
+  		<GPSSensorToROS>
+  			<name>gps_sensor</name>
+  			<topic>/${ns}/gps</topic>
+  			<rate>1</rate>
+  		</GPSSensorToROS>
+  		<DVLSensorToROS>
+  			<name>dvl_sensor</name>
+  			<topic>/${ns}/dvl</topic>
+  			<rate>5</rate>
+  		</DVLSensorToROS>
+  		<RangeImageSensorToROSImage>
+  			<cameraName>depth_camera</cameraName>
+  			<imageTopic> /${ns}/rangecamera </imageTopic>
+  			<infoTopic> /${ns}/rangecamera_info </infoTopic>
+  		</RangeImageSensorToROSImage>
+  		<multibeamSensorToLaserScan>
+  			<name>multibeam</name>
+  			<topic>/${ns}/multibeam</topic>
+  		</multibeamSensorToLaserScan>
+  		<SimulatedDeviceROS>
+  			<echoROS>
+  				<name>g500_echo1</name>
+  				<topic>/${ns}/echo1</topic>
+  				<rate>1</rate>
+  			</echoROS>
+  		</SimulatedDeviceROS>
+  		<contactSensorToROS>
+  			<name>${vehicle_name}</name>
+  			<topic>/${ns}/contactSensor</topic>
+  			<rate> 100 </rate>
+  		</contactSensorToROS>
+  		<echoROS>
+  			<name>g500_echo2</name>
+  			<topic>/${ns}/echo2</topic>
+  			<rate>1</rate>
+  		</echoROS>
+  		<ForceSensorROS>
+  			<name>ForceG500</name>
+  			<topic>/${ns}/ForceSensor</topic>
+  			<rate>100</rate>
+  		</ForceSensorROS>
+  	</rosInterfaces>
+  </xacro:macro>
 </robot>

File: uwsim/data/scenes/params_base.xacro (robot description, xacro)
@@ -2,3 +2,5 @@
 <robot>
 	<property name="M_PI" value="3.1415926535897931" />
+	<property name="ns" value="uwsim" />
+	<property name="vehicle_name" value="girona500" />
 </robot>
